File: pcb/PiCon/picon_v0_0.sch (EAGLE design)
At the start: 3 parts

Commit message: Misc changes
Parts:
- added JP3: (no value), SparkFun-Connectors:M04PTH
- added U$1: CD4068BDIL28-3, Long-Island-Ice-Tea:CD4068BDIL28-3
Changed lines of the file:
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@@
 <part name="JP2" library="SparkFun-Connectors" deviceset="M10" device="&quot;"/>
 <part name="QG1" library="crystal" deviceset="TC46" device="" technology="C"/>
+<part name="U$1" library="Long-Island-Ice-Tea" deviceset="CD4068B" device="DIL28-3"/>
+<part name="JP3" library="SparkFun-Connectors" deviceset="M04" device="PTH"/>
 </parts>
 <sheets>
@@
 <instance part="JP2" gate="G$1" x="134.62" y="45.72"/>
 <instance part="QG1" gate="G$1" x="10.16" y="86.36"/>
+<instance part="U$1" gate="G$1" x="73.66" y="76.2"/>
+<instance part="JP3" gate="G$1" x="124.46" y="78.74"/>
 </instances>
 <busses>
