File: pcb/Vallhalla/v0.1/valhalla_v0.1.sch (EAGLE design)
At the start: 15 parts, among them J1 POWER_JACKPTH, U1 LM317, U2 TLC5940-NT

Commit message: Misc changes based on availability of components
Parts:
- added R3: 120, SparkFun:RESISTORPTH1
- added R6: TRIMPOTPTH, SparkFun-Electromechanical:TRIMPOTPTH
- R1: value 240 -> 120
- R4: value 330 -> 390
- R5: value (none) -> 1.2K
Connections:
- new net N$22: R1.1, R3.2
- new net N$24: R2.2, R3.1, U1.ADJ
- net GND: now also R6.CCW; no longer R5.1
- net N$5: now also R5.1, R6.WIPER; no longer R1.1, R2.2, U1.ADJ
Other:
- moved on the sheet: D1, R2
Changed lines of the file:
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@@
 <part name="R2" library="SparkFun" deviceset="RESISTOR" device="PTH1" value="390"/>
 <part name="C1" library="SparkFun" deviceset="CAP_POL" device="PTH1" value="100uF"/>
-<part name="R1" library="SparkFun" deviceset="RESISTOR" device="PTH1" value="240"/>
-<part name="R4" library="SparkFun" deviceset="RESISTOR" device="PTH1" value="330"/>
+<part name="R1" library="SparkFun" deviceset="RESISTOR" device="PTH1" value="120"/>
+<part name="R4" library="SparkFun" deviceset="RESISTOR" device="PTH1" value="390"/>
 <part name="C2" library="SparkFun" deviceset="CAP_POL" device="PTH2" value="10uF"/>
 <part name="LED2" library="SparkFun-Nate" deviceset="LED" device="5MM" value="Power"/>
@@
 <part name="JP2" library="SparkFun-Connectors" deviceset="M16" device="PTH"/>
 <part name="GND9" library="SparkFun" deviceset="GND" device=""/>
-<part name="R5" library="SparkFun-Resistors" deviceset="RESISTOR" device="PTH-1/2W"/>
+<part name="R5" library="SparkFun-Resistors" deviceset="RESISTOR" device="PTH-1/2W" value="1.2K"/>
+<part name="R3" library="SparkFun" deviceset="RESISTOR" device="PTH1" value="120"/>
+<part name="R6" library="SparkFun-Electromechanical" deviceset="TRIMPOT" device="PTH"/>
 </parts>
 <sheets>
@@
 <instances>
 <instance part="S1" gate="1" x="27.94" y="73.66"/>
-<instance part="R2" gate="G$1" x="68.58" y="48.26" rot="R90"/>
+<instance part="R2" gate="G$1" x="68.58" y="33.02" rot="R90"/>
 <instance part="C1" gate="G$1" x="58.42" y="66.04"/>
 <instance part="R1" gate="G$1" x="78.74" y="63.5" rot="R90"/>
@@
 <instance part="C2" gate="G$1" x="86.36" y="66.04"/>
 <instance part="LED2" gate="G$1" x="109.22" y="53.34"/>
-<instance part="GND1" gate="1" x="86.36" y="27.94"/>
+<instance part="GND1" gate="1" x="86.36" y="20.32"/>
 <instance part="GND3" gate="1" x="109.22" y="43.18"/>
 <instance part="GND5" gate="1" x="58.42" y="55.88"/>
@@
 <instance part="J1" gate="G$1" x="0" y="66.04"/>
 <instance part="JP5" gate="G$1" x="20.32" y="68.58" rot="R180"/>
-<instance part="D1" gate="G$1" x="38.1" y="71.12" smashed="yes">
-<attribute name="NAME" x="36.83" y="73.1266" size="1.778" layer="95"/>
-<attribute name="VALUE" x="33.274" y="67.31" size="1.778" layer="96"/>
+<instance part="D1" gate="G$1" x="43.18" y="71.12" smashed="yes">
+<attribute name="NAME" x="41.91" y="73.1266" size="1.778" layer="95"/>
+<attribute name="VALUE" x="38.354" y="67.31" size="1.778" layer="96"/>
 </instance>
 <instance part="GND7" gate="1" x="10.16" y="60.96"/>
@@
 <instance part="GND2" gate="1" x="33.02" y="-55.88"/>
 <instance part="JP2" gate="G$1" x="152.4" y="-22.86" rot="R180"/>
-<instance part="GND9" gate="1" x="83.82" y="-55.88"/>
+<instance part="GND9" gate="1" x="83.82" y="-66.04"/>
 <instance part="R5" gate="G$1" x="68.58" y="-38.1" rot="R90"/>
+<instance part="R3" gate="G$1" x="78.74" y="50.8" rot="R90"/>
+<instance part="R6" gate="R?" x="68.58" y="-53.34" smashed="yes" rot="R90">
+<attribute name="NAME" x="67.0814" y="-64.77" size="1.778" layer="95" rot="R90"/>
+<attribute name="VALUE" x="71.882" y="-59.69" size="1.778" layer="96" rot="R90"/>
+</instance>
 </instances>
 <busses>
@@
 <net name="GND" class="0">
 <segment>
-<wire x1="86.36" y1="30.48" x2="86.36" y2="38.1" width="0.1524" layer="91"/>
 <pinref part="GND1" gate="1" pin="GND"/>
 <pinref part="C2" gate="G$1" pin="-"/>
-<wire x1="86.36" y1="38.1" x2="86.36" y2="60.96" width="0.1524" layer="91"/>
-<wire x1="68.58" y1="43.18" x2="68.58" y2="38.1" width="0.1524" layer="91"/>
+<wire x1="86.36" y1="22.86" x2="86.36" y2="25.4" width="0.1524" layer="91"/>
 <pinref part="R2" gate="G$1" pin="1"/>
-<wire x1="68.58" y1="38.1" x2="86.36" y2="38.1" width="0.1524" layer="91"/>
-<junction x="86.36" y="38.1"/>
+<wire x1="86.36" y1="25.4" x2="86.36" y2="60.96" width="0.1524" layer="91"/>
+<wire x1="68.58" y1="27.94" x2="68.58" y2="30.48" width="0.1524" layer="91"/>
+<wire x1="68.58" y1="27.94" x2="68.58" y2="25.4" width="0.1524" layer="91"/>
+<wire x1="68.58" y1="25.4" x2="86.36" y2="25.4" width="0.1524" layer="91"/>
+<junction x="86.36" y="25.4"/>
 </segment>
 <segment>
@@
 <pinref part="GND9" gate="1" pin="GND"/>
 <wire x1="86.36" y1="-38.1" x2="83.82" y2="-38.1" width="0.1524" layer="91"/>
-<wire x1="83.82" y1="-38.1" x2="83.82" y2="-45.72" width="0.1524" layer="91"/>
-<pinref part="R5" gate="G$1" pin="1"/>
-<wire x1="83.82" y1="-45.72" x2="83.82" y2="-53.34" width="0.1524" layer="91"/>
-<wire x1="68.58" y1="-43.18" x2="68.58" y2="-45.72" width="0.1524" layer="91"/>
-<wire x1="68.58" y1="-45.72" x2="83.82" y2="-45.72" width="0.1524" layer="91"/>
-<junction x="83.82" y="-45.72"/>
-</segment>
-</net>
-<net name="N$5" class="0">
-<segment>
-<wire x1="68.58" y1="53.34" x2="68.58" y2="55.88" width="0.1524" layer="91"/>
-<wire x1="68.58" y1="55.88" x2="68.58" y2="63.5" width="0.1524" layer="91"/>
-<wire x1="78.74" y1="58.42" x2="78.74" y2="55.88" width="0.1524" layer="91"/>
-<wire x1="78.74" y1="55.88" x2="68.58" y2="55.88" width="0.1524" layer="91"/>
-<junction x="68.58" y="55.88"/>
-<pinref part="R2" gate="G$1" pin="2"/>
-<pinref part="R1" gate="G$1" pin="1"/>
-<pinref part="U1" gate="G$1" pin="ADJ"/>
+<wire x1="83.82" y1="-38.1" x2="83.82" y2="-60.96" width="0.1524" layer="91"/>
+<pinref part="R6" gate="R?" pin="CCW"/>
+<wire x1="83.82" y1="-60.96" x2="83.82" y2="-63.5" width="0.1524" layer="91"/>
+<wire x1="68.58" y1="-58.42" x2="68.58" y2="-60.96" width="0.1524" layer="91"/>
+<wire x1="68.58" y1="-60.96" x2="83.82" y2="-60.96" width="0.1524" layer="91"/>
+<junction x="83.82" y="-60.96"/>
 </segment>
 </net>
@@
 <pinref part="RAW" gate="1" pin="VCC"/>
 <pinref part="D1" gate="G$1" pin="C"/>
-<wire x1="40.64" y1="71.12" x2="58.42" y2="71.12" width="0.1524" layer="91"/>
+<wire x1="45.72" y1="71.12" x2="58.42" y2="71.12" width="0.1524" layer="91"/>
 </segment>
 </net>
@@
 <net name="N$2" class="0">
 <segment>
-<wire x1="33.02" y1="71.12" x2="35.56" y2="71.12" width="0.1524" layer="91"/>
+<wire x1="33.02" y1="71.12" x2="40.64" y2="71.12" width="0.1524" layer="91"/>
 <pinref part="D1" gate="G$1" pin="A"/>
 <pinref part="S1" gate="1" pin="S"/>
@@
 </segment>
 </net>
+<net name="N$22" class="0">
+<segment>
+<pinref part="R1" gate="G$1" pin="1"/>
+<pinref part="R3" gate="G$1" pin="2"/>
+<wire x1="78.74" y1="58.42" x2="78.74" y2="55.88" width="0.1524" layer="91"/>
+</segment>
+</net>
+<net name="N$24" class="0">
+<segment>
+<pinref part="R3" gate="G$1" pin="1"/>
+<wire x1="78.74" y1="45.72" x2="78.74" y2="43.18" width="0.1524" layer="91"/>
+<wire x1="68.58" y1="38.1" x2="68.58" y2="43.18" width="0.1524" layer="91"/>
+<pinref part="R2" gate="G$1" pin="2"/>
+<pinref part="U1" gate="G$1" pin="ADJ"/>
+<wire x1="68.58" y1="43.18" x2="68.58" y2="63.5" width="0.1524" layer="91"/>
+<wire x1="78.74" y1="43.18" x2="68.58" y2="43.18" width="0.1524" layer="91"/>
+<junction x="68.58" y="43.18"/>
+</segment>
+</net>
+<net name="N$5" class="0">
+<segment>
+<pinref part="R5" gate="G$1" pin="1"/>
+<wire x1="68.58" y1="-43.18" x2="60.96" y2="-43.18" width="0.1524" layer="91"/>
+<wire x1="60.96" y1="-43.18" x2="60.96" y2="-53.34" width="0.1524" layer="91"/>
+<pinref part="R6" gate="R?" pin="WIPER"/>
+<wire x1="60.96" y1="-53.34" x2="63.5" y2="-53.34" width="0.1524" layer="91"/>
+</segment>
+</net>
